Commit message: Add full autonomous navigation stack with tests and RViz2
Planning:
- Extract pure astar() into planning.py with inflate_obstacles() and
  prune_path(); planner now replans from the robot's current grid position
  and skips already-reached checkpoints after each /current_checkpoint event
- Obstacle inflation (configurable radius, default 1 cell) with start/goal
  exemption; fallback to un-inflated plan if inflation blocks the goal
- Collinear waypoint pruning reduces grid staircases to straight-line segments

Control:
- Replace proportional heading controller with Pure Pursuit (lookahead 1.5 m)
- Adaptive speed scaling via speed_scale_from_scan(): full speed >2 m clearance,
  linear ramp to zero at STOP_DIST (0.6 m)
- Emergency stop from /scan forward arc (±45°), independent of planner
- Stuck detection: no movement >8 cm in 6 s → publish /replan_request and reset
- Broadcast odom→base_link TF on every /odom so full TF tree is live in RViz2

New node — scan_occupancy:
- Converts /scan hits to grid cells using robot pose from /odom
- 3 s decay window; publishes /map/scan_obstacles at 5 Hz
- Pure function scan_hits_to_grid() exposed for unit testing

New topics:
  /current_checkpoint  Int32   — 1-indexed checkpoint reached event
  /mission_complete    Bool    — True when all checkpoints done
  /replan_request      Empty   — forces immediate replan
  /checkpoint_markers  MarkerArray — green→grey spheres + labels in RViz2
  /lookahead_marker    Marker  — orange sphere at Pure Pursuit target
  /map/scan_obstacles  GridCells — live lidar obstacle layer

Launch:
- obstacles_csv / checkpoints_csv launch args — substitute any CSV at launch
  time without rebuilding; default to bundled config/
- no_rviz:=true for headless / CI runs
- Static map→odom identity TF publisher
- ignition-gazebo-sensors-system plugin for GPU lidar
- /scan bridged via ros_gz_bridge

URDF:
- Add laser_link (front x=0.20 z=0.10) with 360° gpu_lidar sensor,
  10 Hz, 0.1–12 m range, Gaussian noise σ=0.01 m

Tests (85 total, colcon test + pytest):
- test_astar.py        — A* correctness, obstacle avoidance, path quality
- test_planning_utils.py — inflate_obstacles, prune_path
- test_controller_math.py — normalise, yaw_from_quat, heading_error,
                            compute_cmd, pure pursuit, speed_scale_from_scan
- test_scan_math.py    — scan_hits_to_grid coordinate transform and filtering

File: src/av_sim/urdf/robot.urdf (robot description, URDF)
Before this commit: robot diff_drive_robot, 4 links, 3 joints
Links:
- added link laser_link, mass 0.1; collision cylinder length=0.04 radius=0.04; visual cylinder length=0.04 radius=0.04
Joints:
- added joint laser_joint: type fixed, parent base_link, child laser_link, origin xyz=0.20 0.0 0.10 rpy=0 0 0

Commit message: feat: URDF — Gazebo Classic diff_drive + CPU ray sensor (no gpu_lidar)

File: src/av_sim/urdf/robot.urdf (robot description, URDF)
Before this commit: robot diff_drive_robot, 4 links, 3 joints
Links:
- removed link caster_wheel
- added link caster_link, mass 0.1; collision sphere radius=0.04; visual sphere radius=0.04
- added link laser_link; visual cylinder length=0.04 radius=0.03
- link base_link: mass 10.0 -> 5.0; geometry collision box size=0.4 0.3 0.1; visual box size=0.4 0.3 0.1
- link left_wheel: mass 1.0 -> 0.5; geometry collision cylinder length=0.04 radius=0.1; visual cylinder length=0.04 radius=0.1
- link right_wheel: mass 1.0 -> 0.5; geometry collision cylinder length=0.04 radius=0.1; visual cylinder length=0.04 radius=0.1
Joints:
- added joint laser_joint: type fixed, parent base_link, child laser_link, origin xyz=0 0 0.1 rpy=0 0 0
- joint caster_joint: child caster_wheel -> caster_link; origin xyz=-0.20 0.0 -0.125 rpy=0 0 0 -> xyz=-0.15 0 -0.07 rpy=0 0 0
- joint left_wheel_joint: origin xyz=0.0 0.175 -0.075 rpy=-1.5708 0.0 0.0 -> xyz=0 0.17 -0.025 rpy=-1.5708 0 0
- joint right_wheel_joint: origin xyz=0.0 -0.175 -0.075 rpy=-1.5708 0.0 0.0 -> xyz=0 -0.17 -0.025 rpy=-1.5708 0 0

Commit message: fix: correct chassis inertia tensor and caster joint z offset

File: src/av_sim/urdf/robot.urdf (robot description, URDF)
Before this commit: robot av_robot, 5 links, 4 joints
Joints:
- joint caster_joint: origin xyz=-0.15 0 -0.07 rpy=0 0 0 -> xyz=-0.15 0 -0.085 rpy=0 0 0
